Commit message: r2d2 and launch file with nodes and remap

File: src/vlad_r2d2/urdf/r2d2.urdf (robot description, URDF)
Before this commit: robot physics, 17 links, 16 joints
Joints:
- joint lenstobox: limit (none) -> lower=-0.02 upper=0.02 effort=10 velocity=0.5; origin xyz=0.025 0 0 rpy=0 1.57075 0 -> xyz=0 0 0 rpy=0 0 0; type fixed -> prismatic

File: src/vlad_r2d2/urdf/r2d2.urdf.xacro (robot description, xacro)
@@ -219,4 +219,5 @@
       </geometry>
       <material name="black"/>
+      <origin xyz="0 0 0" rpy="0 ${pi/2} 0"/>
     </visual>
     <collision>
@@ -224,11 +225,20 @@
         <cylinder length="0.05" radius="0.04"/>
       </geometry>
+      <origin xyz="0.04 0 0" rpy="0 ${pi/2} 0"/>
     </collision>
     <xacro:default_inertial mass="1"/>
   </link>
-  <joint name="lenstobox" type="fixed">
+  <joint name="lenstobox" type="prismatic">
     <parent link="box"/>
     <child link="lens"/>
-    <origin rpy="0 1.57075 0" xyz="0.025 0 0"/>
+    <limit effort="10" lower="-0.02" upper="0.02" velocity="0.5"/>
+    <origin xyz="0 0 0" rpy="0 0 0"/>
+  </joint>
+  <link name="base_footprint">
+  </link>
+  <joint name="basefloor" type="fixed">
+  	<parent link="base_footprint"/>
+  	<child link="base_link"/>
+  	<origin xyz="0 0 ${bodylen/2+0.1+wheeldiam}"/>
   </joint>
 </robot>
